File: rusty-tracker.kicad_sch (KiCad schematic)
At the start: 174 parts, among them J1 SIM8051-6-0-14-01-X, J2 USB_C_Receptacle_USB2.0, J3 NFC, J4 tag-connect-swd, J5 Battery Connector, Q1 BC846, Q2 BC846, SW1 SW_Push, T1 Tab, T2 Tab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

Commit message: Added buzzer
Parts:
- added BZ1: Buzzer, buzzers:AST0927, symbol Device:Buzzer
- added D10: 1N4148, passive:D_0402_DFN1006, symbol Device:D_Small
- added Q3: BC846, sot:SOT-323, symbol Device:Q_NPN_BEC
- added R38: 470, passive:R_0402, symbol Device:R_Small
Connections:
- net +BATT: now also BZ1.1 (-), D10.1 (K)
- net GND: now also Q3.2 (E)
- net BUZ: now reaches U2.B17 (P1.12)
- net BUZ: now also R38.1
- new net: BZ1.2 (+), D10.2 (A), Q3.3 (C)
- new net: Q3.1 (B), R38.2
- no-connect marks 58 -> 57
