File: rusty-tracker.kicad_sch (KiCad schematic)
At the start: 176 parts, among them J1 SIM8051-6-0-14-01-X, J2 USB_C_Receptacle_USB2.0, J3 NFC, J4 tag-connect-swd, J5 Battery Connector, J6 Conn_01x01, J7 Conn_01x01, Q1 RUM002N02T2L, Q2 RUM002N02T2L, Q3 RUM002N02T2L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

Commit message: MFPNs added
Parts:
- Ant3: MFPN (none) -> P822602
- BZ1: MFPN (none) -> AST0927MW-03TRQ
- C6, C7: Tolerance 1% -> (none)
- D1, D10: MFPN (none) -> 1N4148WL2-TP
- D8: MFPN (none) -> ESD122DMYR
- FB1, FB2: MFPN (none) -> BLM18EG221SN1D
- J1: MFPN (none) -> SIM8051-6-0-14-01-A
- J2: MFPN (none) -> USB4105-GF-A
- SW1: MFPN (none) -> EVQ-P2602W
- U1: MFPN (none) -> SARA-R422M10S-01B
- U10, U11, U9: MFPN (none) -> MM8130-2600
- U2: MFPN (none) -> NRF52840-QIAA
- U5: MFPN (none) -> MCP73833-AMI/MF
- U8: MFPN (none) -> B39242B8328P810
Changed lines of the file:
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@@
       (effects (font (size 1.27 1.27)) hide)
     )
+    (property "MFPN" "AST0927MW-03TRQ" (at 384.81 191.77 0)
+      (effects (font (size 1.27 1.27)) hide)
+    )
     (pin "1")
     (pin "2")
@@
       (effects (font (size 1.27 1.27)) hide)
     )
+    (property "MFPN" "1N4148WL2-TP" (at 389.89 191.77 0)
+      (effects (font (size 1.27 1.27)) hide)
+    )
     (pin "1")
     (pin "2")
@@
       (effects (font (size 1.27 1.27)))
     )
-    (property "Tolerance" "1%" (at 275.59 176.53 0)
+    (property "Tolerance" "" (at 275.59 176.53 0)
       (effects (font (size 1.524 1.524)) hide)
     )
@@
       (effects (font (size 1.27 1.27)) hide)
     )
+    (property "MFPN" "ESD122DMYR" (at 182.88 245.11 0)
+      (effects (font (size 1.27 1.27)) hide)
+    )
     (pin "1")
     (pin "2")
@@
       (effects (font (size 1.27 1.27)) hide)
     )
+    (property "MFPN" "MM8130-2600" (at 73.66 259.08 0)
+      (effects (font (size 1.27 1.27)) hide)
+    )
     (pin "1")
     (pin "2")
@@
       (effects (font (size 1.27 1.27)) hide)
     )
+    (property "MFPN" "NRF52840-QIAA" (at 320.04 162.56 0)
+      (effects (font (size 1.27 1.27)) hide)
+    )
     (pin "A10")
     (pin "A12")
@@
       (effects (font (size 1.27 1.27)) hide)
     )
+    (property "MFPN" "EVQ-P2602W" (at 388.62 226.06 0)
+      (effects (font (size 1.27 1.27)) hide)
+    )
     (pin "1")
     (pin "2")
@@
       (effects (font (size 1.27 1.27)) hide)
     )
+    (property "MFPN" "USB4105-GF-A" (at 127 237.49 0)
+      (effects (font (size 1.27 1.27)) hide)
+    )
     (pin "A1")
     (pin "A12")
@@
       (effects (font (size 1.27 1.27)) hide)
     )
+    (property "MFPN" "1N4148WL2-TP" (at 389.89 162.56 0)
+      (effects (font (size 1.27 1.27)) hide)
+    )
     (pin "1")
     (pin "2")
@@
       (effects (font (size 1.27 1.27)) hide)
     )
+    (property "MFPN" "MM8130-2600" (at 40.64 214.63 0)
+      (effects (font (size 1.27 1.27)) hide)
+    )
     (pin "1")
     (pin "2")
@@
       (effects (font (size 1.27 1.27)) hide)
     )
+    (property "MFPN" "B39242B8328P810" (at 101.6 163.83 0)
+      (effects (font (size 1.27 1.27)) hide)
+    )
     (pin "1")
     (pin "2")
@@
       (effects (font (size 1.27 1.27)))
     )
+    (property "MFPN" "P822602" (at 99.06 214.63 0)
+      (effects (font (size 1.27 1.27)) hide)
+    )
     (pin "1")
     (pin "2")
@@
       (effects (font (size 1.27 1.27)) hide)
     )
-    (property "MFPN" "" (at 271.78 25.4 0)
+    (property "MFPN" "MCP73833-AMI/MF" (at 271.78 25.4 0)
       (effects (font (size 1.27 1.27)) hide)
     )
@@
       (effects (font (size 1.27 1.27)))
     )
-    (property "Tolerance" "1%" (at 283.21 176.53 0)
+    (property "Tolerance" "" (at 283.21 176.53 0)
       (effects (font (size 1.524 1.524)) hide)
     )
@@
       (effects (font (size 1.27 1.27)) hide)
     )
+    (property "MFPN" "SARA-R422M10S-01B" (at 67.31 31.75 0)
+      (effects (font (size 1.27 1.27)) hide)
+    )
     (pin "1")
     (pin "10")
@@
       (effects (font (size 1.27 1.27)) hide)
     )
+    (property "MFPN" "BLM18EG221SN1D" (at 115.57 133.35 0)
+      (effects (font (size 1.27 1.27)) hide)
+    )
     (pin "1")
     (pin "2")
@@
       (effects (font (size 1.27 1.27)) hide)
     )
+    (property "MFPN" "BLM18EG221SN1D" (at 180.34 222.25 0)
+      (effects (font (size 1.27 1.27)) hide)
+    )
     (pin "1")
     (pin "2")
@@
       (effects (font (size 1.27 1.27)) hide)
     )
+    (property "MFPN" "MM8130-2600" (at 66.04 166.37 0)
+      (effects (font (size 1.27 1.27)) hide)
+    )
     (pin "1")
     (pin "2")
@@
       (effects (font (size 1.27 1.27)) hide)
     )
+    (property "MFPN" "SIM8051-6-0-14-01-A" (at 212.09 172.72 0)
+      (effects (font (size 1.27 1.27)) hide)
+    )
